Commit message: frame rellationships change
change the tf relationships to
base_link -> base_footprint

File: urdf/test.urdf (robot description, URDF)
Before this commit: robot test_robot, 6 links, 5 joints
Joints:
- removed joint base_footprint_to_base_link
- added joint base_link_to_base_footprint: type fixed, parent base_link, child base_footprint

File: urdf/test.xacro (robot description, xacro)
@@ -139,7 +139,7 @@
     <!--###########ジョイントの作成##########-->
     <!--base_footprintとbase_link-->
-    <joint name="base_footprint_to_base_link" type="fixed">
-        <parent link="base_footprint" />
-        <child link="base_link" />
+    <joint name="base_link_to_base_footprint" type="fixed">
+        <parent link="base_link" />
+        <child link="base_footprint" />
     </joint>
     <!--LiDARとbase_link-->
@@ -188,5 +188,5 @@
         <publish_tf>true</publish_tf>
         <odometry_frame>odom</odometry_frame>
-        <robot_base_frame>base_footprint</robot_base_frame>
+        <robot_base_frame>base_link</robot_base_frame>
     </plugin>
     </gazebo>

Commit message: self_driving_ver.1
Integrating autonomous navigation into my robot

File: urdf/test.urdf (robot description, URDF)
Before this commit: robot test_robot, 6 links, 5 joints
Joints:
- joint base_link_to_caster_wheel: axis 1 0 0 -> 0 1 0; origin xyz=0 0.25 0.05 -> xyz=-0.25 0 0.05
- joint base_link_to_left_wheel: axis 1 0 0 -> 0 1 0; origin xyz=-0.525 0 0.1 -> xyz=0 0.525 0.1
- joint base_link_to_right_wheel: axis 1 0 0 -> 0 1 0; origin xyz=0.525 0 0.1 -> xyz=0 -0.525 0.1

File: urdf/test.xacro (robot description, xacro)
@@ -63,5 +63,5 @@
             <cylinder length="${wheellen}" radius="${wheelrad}"/>
         </geometry>
-        <origin rpy="0 1.57075 0" xyz="0 0 0"/>
+        <origin rpy="1.57075 0 0" xyz="0 0 0"/>
         <material name="black"/>
         </visual>
@@ -70,8 +70,8 @@
                 <cylinder length="${wheellen}" radius="${wheelrad}"/>
             </geometry>
-            <origin rpy="0 1.57075 0" xyz="0 0 0"/>
-        </collision>
-        <inertial>
-            <origin rpy="0 1.57075 0" xyz="0 0 0"/>
+            <origin rpy="1.57075 0 0" xyz="0 0 0"/>
+        </collision>
+        <inertial>
+            <origin rpy="1.57075 0 0" xyz="0 0 0"/>
             <mass value="1"/>
             <inertia ixx="${1/4*1*wheelrad*wheelrad+1/12*2*wheellen}" ixy="0.0" ixz="0.0" iyy="${1/4*1*wheelrad*wheelrad+1/12*2*wheellen}" iyz="0.0" izz="${1/2*1*wheelrad*wheelrad}"/>
@@ -89,5 +89,5 @@
             <cylinder length="${wheellen}" radius="${wheelrad}"/>
         </geometry>
-        <origin rpy="0 1.57075 0" xyz="0 0 0"/>
+        <origin rpy="1.57075 0 0" xyz="0 0 0"/>
         <material name="black"/>
         </visual>
@@ -96,8 +96,8 @@
                 <cylinder length="${wheellen}" radius="${wheelrad}"/>
             </geometry>
-            <origin rpy="0 1.57075 0" xyz="0 0 0"/>
-        </collision>
-        <inertial>
-            <origin rpy="0 1.57075 0" xyz="0 0 0"/>
+            <origin rpy="1.57075 0 0" xyz="0 0 0"/>
+        </collision>
+        <inertial>
+            <origin rpy="1.57075 0 0" xyz="0 0 0"/>
             <mass value="1"/>
             <inertia ixx="${1/4*1*wheelrad*wheelrad+1/12*2*wheellen}" ixy="0.0" ixz="0.0" iyy="${1/4*1*wheelrad*wheelrad+1/12*2*wheellen}" iyz="0.0" izz="${1/2*2*wheelrad*wheelrad}"/>
@@ -115,5 +115,5 @@
             <sphere radius="0.05"/>
         </geometry>
-        <origin rpy="0 0 0" xyz="0 0 0"/>
+        <origin  xyz="0 0 0"/>
         <material name="black"/>
         </visual>
@@ -122,13 +122,12 @@
                 <sphere radius="0.05"/>
             </geometry>
-            <origin rpy="0 0 0" xyz="0 0 0"/>
-        </collision>
-        <inertial>
-            <origin rpy="0 1.57075 0" xyz="0 0 0"/>
+            <origin xyz="0 0 0"/>
+        </collision>
+        <inertial>
+            <origin  xyz="0 0 0"/>
             <mass value="1"/>
             <inertia ixx="${2/5*1*0.05*0.05}" ixy="0" ixz="0" iyy="${2/5*1*0.05*0.05}" iyz="0" izz="${2/5*1*0.05*0.05}"/>
         </inertial>
     </link>
-    <!--
     <gazebo reference="caster_wheel">
         <material>
@@ -136,5 +135,4 @@
         </material>
     </gazebo>
-    -->
     <!--###########ジョイントの作成##########-->
     <!--base_footprintとbase_link-->
@@ -154,6 +152,6 @@
         <parent link="base_link"/>
         <child link="right_wheel"/>
-        <origin xyz = "${baserad+wheellen/2} 0 ${wheelrad}"/>
-        <axis xyz = "1 0 0"/>
+        <origin xyz = "0 ${-(baserad+wheellen/2)} ${wheelrad}"/>
+        <axis xyz = "0 1 0"/>
     </joint>
     <!--base_linkとleft_wheel-->
@@ -161,6 +159,6 @@
         <parent link="base_link"/>
         <child link="left_wheel"/>
-        <origin xyz = "${-(baserad+wheellen/2)} 0 ${wheelrad}"/>
-        <axis xyz = "1 0 0"/>
+        <origin xyz = "0 ${baserad+wheellen/2} ${wheelrad}"/>
+        <axis xyz = "0 1 0"/>
     </joint>
     <!--base_linkとcaster_wheel-->
@@ -168,6 +166,6 @@
         <parent link="base_link"/>
         <child link="caster_wheel"/>
-        <origin xyz = "0 0.25 0.05"/>
-        <axis xyz = "1 0 0"/>
+        <origin xyz = "-0.25 0 0.05"/>
+        <axis xyz = "0 1 0"/>
     </joint>
     <gazebo>
@@ -177,12 +175,12 @@
         <right_joint>base_link_to_right_wheel</right_joint>
         <!-- kinematics -->
-        <wheel_separation>1</wheel_separation>
+        <wheel_separation>1.05</wheel_separation>
         <wheel_diameter>0.1</wheel_diameter>
         <!-- limits -->
-        <max_wheel_torque>10</max_wheel_torque>
+        <max_wheel_torque>20</max_wheel_torque>
         <max_wheel_acceleration>1.0</max_wheel_acceleration>
         <!-- output -->
-        <publish_odom>true</publish_odom>
-        <publish_odom_tf>true</publish_odom_tf>
+        <publish_odom>True</publish_odom>
+        <publish_odom_tf>True</publish_odom_tf>
         <publish_wheel_tf>false</publish_wheel_tf>
         <publish_tf>true</publish_tf>

Commit message: some revisions

File: urdf/test.urdf (robot description, URDF)
Before this commit: robot test_robot, 6 links, 5 joints
Joints:
- joint base_link_to_LiDAR: origin xyz=0 0 0.5750000000000001 -> xyz=0.5 0 0.07500000000000001

File: urdf/test.xacro (robot description, xacro)
@@ -145,5 +145,5 @@
         <parent link="base_link"/>
         <child link="LiDAR"/>
-        <origin xyz = "0 0 ${baselen+0.05+0.05/2}"/>
+        <origin xyz = "${baserad} 0 ${0.05+0.05/2}"/>
     <axis xyz = "0 0 1"/>
     </joint>
@@ -200,6 +200,6 @@
                         <samples>360</samples>
                         <resolution>1.0</resolution>
-                        <min_angle>0.0</min_angle>
-                        <max_angle>6.28</max_angle>
+                        <min_angle>4.71</min_angle>
+                        <max_angle>7.85</max_angle>
                     </horizontal>
                 </scan>
